File: pcb/m365_esp32.sch (EAGLE design)
At the start: 45 parts, among them J2 105133-0011, Q1 32768kHz, T2 BCX19SMD

Commit message: Placed the buttons, center button multiplexer, usb interface, 3v3 regulator
Parts:
- removed U$12, U$13, U$14, U$15, U$16: KSEK43J, my-lib:KSEK43J
- added ACCEL, BRK: (no value), SparkFun-Connectors:CONN_03LONGPADS
- added C10, C15, C22, C8: 22u, eagle-ltspice:CC0603
- added C11, C12, C13, C14, C21: 0.1uF, eagle-ltspice:CC0402
- added CENTER, DOWN, LEFT, RIGHT, UP: KSEK43J, my-lib:KSEK43J
- added D1, D3, D4: SMAFJ75A, my-lib:SMAFJ75A
- added J1: (no value), SparkFun-Connectors:CONN_04LONGPADS
- added LED: (no value), SparkFun-Connectors:CONN_02PTH3
- added R10, R12: 866k, eagle-ltspice:RR0402
- added R11: 180k, eagle-ltspice:RR0402
- added R9: 6.65k, eagle-ltspice:RR0402
- added T1: L2N7002DW1T1G, nxp_60_1_1:2N7002PS
- added U$7: UZ1085L-33-TN3-R, my-lib:UZ1085L-33-TN3-R
- C4: value 10nF -> 0.1uF
- C7: device eagle-ltspice:CC1210 -> eagle-ltspice:CC0603
- D2: value (none) -> SMAFJ75A; device diode:ZENER-DIODETO236 -> my-lib:SMAFJ75A
- T2: value BCX19SMD -> L2N7002DW1T1G; device transistor-npn:BCX19SMD -> nxp_60_1_1:2N7002PS
Connections:
- removed net VUSB: C4.1, J2.VBUS, R1.1, R2.1, U$2.VCC
- new net 5V_IN: C15.1, C21.1, D3.ANODE, J1.2
- new net 5V_USB: C22.1, C4.1, D4.ANODE, J2.VBUS, R1.1, R2.1, U$2.VCC
- new net BUZZER: T2-2.G
- new net DATA: J1.3
- new net N$10: R9.1, T1-1.D
- new net N$11: CENTER.P$1, D1.CATHODE, T1-2.S
- new net N$12: D2.ANODE, T2-2.D, U$8.-
- new net N$5: R11.2, R12.1, R9.2, T1-2.G
- net 3V3: now also ACCEL.3, BRK.3, C8.1, D2.CATHODE, R10.2, T1-1.G, U$7.VOUT, U$8.+
- net 42V: now also J1.1, R12.2, T1-2.D; no longer D2.C, U$12.P$1
- net 5V: now also C10.1, D3.CATHODE, D4.CATHODE, U$7.VIN
- net A0: now also ACCEL.2
- net A1: now also BRK.2
- net D1: now also D1.ANODE; no longer D2.A
- net D13-SCK: now also C13.2, DOWN.P$1; no longer U$16.P$1
- net D2: now also C14.2, UP.P$1; no longer U$15.P$1
- net D3: now also C11.1, LEFT.P$1; no longer U$13.P$1
- net D4-MOSI: now also C12.1, RIGHT.P$1; no longer U$14.P$1
- net FRONT_LED: now also LED.1
- net GND: now also ACCEL.1, BRK.1, C10.2, C11.2, C12.2, C13.1, C14.1, C15.2, C21.2, C22.2, C8.2, CENTER.P$2, DOWN.P$2, J1.4, LED.2, LEFT.P$2, R10.1, R11.1, RIGHT.P$2, T1-1.S, T2-1.D, T2-1.G, T2-1.S, T2-2.S, U$7.GND, UP.P$2; no longer U$12.P$2, U$13.P$2, U$14.P$2, U$15.P$2, U$16.P$2
Other:
- moved on the sheet: C4, D2, U$8

Commit message: Finished placing all components on the board
Parts:
- added C25: 22u, eagle-ltspice:CC0603
- added C26, C27: 0.1uF, eagle-ltspice:CC0402
- added J3: (no value), SparkFun-Connectors:CONN_06LOCK
Connections:
- net D3 renamed BTN_LEFT
- net D4-MOSI renamed BTN_RIGHT
- removed net A0: ACCEL.2, U$1.SENSOR_VP(GPI36/ADC1:0/RTC0)
- removed net A1: BRK.2, U$1.SENSOR_CAPP(GPI37/ADC1:1/RTC1)
- removed net D0: U$1.GPIO23
- removed net D1: D1.ANODE, U$1.(VSPICLK/HS1_DATA7)GPIO18
- removed net D13-SCK: C13.2, DOWN.P$1, U$1.(ADC2:0/TOUCH0/RTC10/SPIHD)GPIO4
- removed net D14: U$1.(GPIO7/SPI1/HS1_DATA0)SD_DATA0
- removed net D15: U$1.(GPIO8/SPID/HS1_DATA1)SD_DATA1
- removed net D2: C14.2, U$1.(VSPICS0/HS1_DATA6)GPIO5, UP.P$1
- removed net D5-MISO: U$1.(DAC1/ADC2:8/RTC6)GPIO25
- removed net D6: U$1.(DAC2/ADC2:9/RTC7)GPIO26
- removed net D7: U$1.(ADC2:7/TOUCH7/RTC17)GPIO27
- removed net RGB_B: U$1.(GPIO6/SPICLK/HS1_CLK/U1CTS)SD_CLK
- removed net RGB_G: U$1.(GPIO11/SPICSO/HS1_CMD/U1RTS)SD_CMD
- removed net RGB_R: U$1.(GPIO10/SPIWP/HS1_DATA3/U1TX)SD_DATA3
- removed net SCL: U$1.(VSPIWP/HS2_CLK)GPIO22
- removed net SDA: U$1.(VSPIHD/HS2_CMD)GPIO21
- new net BTN_CENTER: C27.1, D1.ANODE, U$1.(VSPICS0/HS1_DATA6)GPIO5
- new net BTN_DOWN: C13.2, DOWN.P$1, U$1.(VSPICLK/HS1_DATA7)GPIO18
- new net BTN_UP: C14.2, U$1.GPIO23, UP.P$1
- net !DTR1: now also J3.6
- net !RTS1: now also J3.2
- net 3V3: now also C25.1, C26.1
- net 5V_USB: now also J3.3
- net A2: now also ACCEL.2
- net A5: now also BRK.2
- net GND: now also C25.2, C26.2, C27.2, J3.1
- net RX0: now also J3.4
- net TX0: now also J3.5
Other:
- note added: "Near Buzzer"
- note added: "Near microUSB"
- moved on the sheet: C11, C12, C13, C14, J1

Commit message: Finished dashboard PCB
Parts:
- removed ACCEL: (no value), SparkFun-Connectors:CONN_03LONGPADS
- removed Q1: 32768kHz, crystal:FC-12M
- removed RX1, TX1: (no value), adafruit:LEDCHIP-LED0603
- added ACC: (no value), SparkFun-Connectors:CONN_03LONGPADS
- added C28, C29, C30, C31: 0.1uF, eagle-ltspice:CC0402
- added D5: SMAFJ75A, my-lib:SMAFJ75A
- added FT231X: FT231XQ-R, FT231XQ-R:FT231XQ-R
- added GOLD_ORB_SM2: OSHWLOGOLOGO5MM, oshw:OSHWLOGOLOGO5MM
- added IC1, IC2: NTS0101GW,125, NTS0101GW_125:NTS0101GW,125
- added LS1: (no value), eagle-ltspice:RR1206
- added M365_CONNECTOR: (no value), SparkFun-Connectors:CONN_05PTH_LONGPADS
- added R13: 16R, eagle-ltspice:RR0402
- added R14, R24, R25, R28, R29, R31: 866k, eagle-ltspice:RR0402
- added R15, R30, R32: 220R, eagle-ltspice:RR0402
- added R17, R20, R23: 86.6R, eagle-ltspice:RR0402
- added R18, R21: 60.4R, eagle-ltspice:RR0402
- added R19, R22, R26, R27: 37.4R, eagle-ltspice:RR0402
- added REG: UZ1085L-33-TN3-R, my-lib:UZ1085L-33-TN3-R
- added T3: L2N7002DW1T1G, nxp_60_1_1:2N7002PS
- added U$10: X321532768KGB2SI, my-lib:X321532768KGB2SI
- added U$11: LH096T-IG11, my-lib:LH096T-IG11
- added USB: 105133-0011, 105133-0011:105133-0011
- C1: value 10u -> 10uF
- C10, C15, C22, C25, C7, C8: value 22u -> 22uF
- C23, C24: value 15pF -> 20pF
- C6: value 100p -> 100pF
- J1: device SparkFun-Connectors:CONN_04LONGPADS -> eagle-ltspice:RR0402
- J2: value 105133-0011 -> (none); device 105133-0011:105133-0011 -> eagle-ltspice:RR0402
- R1, R2: value 499 -> 499R; device resistor:R-EU_R0402 -> eagle-ltspice:RR0402
- R11: device eagle-ltspice:RR0402 -> eagle-ltspice:RR0603
- R3, R4: value 27 -> 27R
- U$2: value FT231XQ-R -> Z3535RGBA; device FT231XQ-R:FT231XQ-R -> my-lib:Z3535RGBA
- U$7: value UZ1085L-33-TN3-R -> Z3535RGBA; device my-lib:UZ1085L-33-TN3-R -> my-lib:Z3535RGBA
- renumbered J3 to PROG
Connections:
- removed net A3: U$1.SENSOR_VN(GPI39/ADC1:3/RTC3)
- removed net A4: U$1.VDET_1(GPI34/ADC1:6)
- removed net CBUS3: RX1.C, U$2.CBUS2
- removed net CBUS4: TX1.C, U$2.CBUS1
- removed net D10: U$1.(GPIO15/ADC2:3/TOUCH3/RTC13/SPICSO/U0RTS)MTDO
- removed net D8: U$1.(GPIO14/ADC2:6/TOUCH6/RTC16/SPICLK)MTMS
- removed net D9: U$1.(GPIO13/ADC2:4/TOUCH4/RTC14/SPID/U0CTS)MTCK
- removed net DATA: J1.3
- new net !TFTRST: U$1.(DAC1/ADC2:8/RTC6)GPIO25, U$11.RESET
- new net BACKLIGHT: R15.1, U$1.(GPIO15/ADC2:3/TOUCH3/RTC13/SPICSO/U0RTS)MTDO
- new net BTN_CONTROL: R30.1
- new net DC: U$1.(DAC2/ADC2:9/RTC7)GPIO26, U$11.RS
- new net LED_K: R13.2, U$11.LEDK
- new net LIGHT_SENS: C30.1, LS1.2, R28.2, U$1.SENSOR_VN(GPI39/ADC1:3/RTC3)
- new net LL_B: R21.1, U$1.(GPIO6/SPICLK/HS1_CLK/U1CTS)SD_CLK
- new net LL_G: R22.1, U$1.(GPIO7/SPI1/HS1_DATA0)SD_DATA0
- new net LL_R: R23.1, U$1.(GPIO8/SPID/HS1_DATA1)SD_DATA1
- new net LR_B: R18.1, U$1.(GPIO11/SPICSO/HS1_CMD/U1RTS)SD_CMD
- new net LR_G: R19.1, U$1.(GPIO10/SPIWP/HS1_DATA3/U1TX)SD_DATA3
- new net LR_R: R20.1, U$1.(GPIO9/SPIHD/HS1_DATA2/U1RX)SD_DATA2
- new net M365_DATA: IC2.B, J2.1, M365_CONNECTOR.3
- new net M365_DATA_3V3: D5.ANODE, IC2.A, J2.2, U$1.(VSPID/HS2_DATA3)GPIO20
- new net M365_LED_DATA: IC1.B, J1.1, M365_CONNECTOR.1
- new net M365_LED_DATA_3V3: IC1.A, J1.2, U$1.(GPIO13/ADC2:4/TOUCH4/RTC14/SPID/U0CTS)MTCK
- new net MOSI: U$1.(ADC2:7/TOUCH7/RTC17)GPIO27, U$11.SDA
- new net N$13: R13.1, T3-1.D
- new net N$14: R14.2, R15.2, T3-1.G
- new net N$15: D5.CATHODE, R17.2
- new net N$16: C29.2, R2.2, U$1.SENSOR_CAPN(GPI38/ADC1:2/RTC2)
- new net N$17: R17.1, U$1.(VSPIQ/HS2_DATA2)GPIO19
- new net N$18: R21.2, U$7.BLUE
- new net N$19: R22.2, U$7.GREEN
- new net N$20: R26.2, U$7.RED
- new net N$21: R18.2, U$2.BLUE
- new net N$22: R19.2, U$2.GREEN
- new net N$23: U$1.(VSPIHD/HS2_CMD)GPIO21
- new net N$25: R27.2, U$2.RED
- new net N$26: R20.2, R27.1
- new net N$27: U$1.(VSPIWP/HS2_CLK)GPIO22
- new net N$28: R10.2, R30.2, T1-1.G
- new net N$29: R32.2, T2-2.G
- new net SCK: U$1.(GPIO14/ADC2:6/TOUCH6/RTC16/SPICLK)MTMS, U$11.SCL
- new net TFTCS: U$1.(GPIO12/ADC2:5/TOUCH5/RTC15/SPIQ)MTDI, U$11.CS
- net !DTR1: now also FT231X.!DTR; no longer U$2.!DTR
- net !RTS1: now also FT231X.!RTS; no longer U$2.!RTS
- net 32K_XP: now also U$10.2; no longer Q1.2
- net 3V3: now also ACC.3, C31.1, IC1.OE, IC1.VCC(A), IC2.OE, IC2.VCC(A), LS1.1, REG.VOUT, U$11.LEDA, U$11.VCC, U$2.VCC, U$7.VCC; no longer ACCEL.3, R10.2, T1-1.G, U$7.VOUT
- net 42V: now also M365_CONNECTOR.5; no longer J1.1
- net 5V: now also IC1.VCC(B), IC2.VCC(B), REG.VIN; no longer U$7.VIN
- net 5V_IN: now also M365_CONNECTOR.2; no longer J1.2
- net 5V_USB: now also FT231X.VCC, USB.VBUS; no longer J2.VBUS, R1.1, R2.1, U$2.VCC
- net A2: now also ACC.2, R2.1, R25.1; no longer ACCEL.2, U$1.SENSOR_CAPN(GPI38/ADC1:2/RTC2)
- net A5: now also R1.1, R24.2; no longer U$1.VDET_2(GPI35/ADC1:7)
- net BTN_CENTER: now also R31.1
- net BUZZER: now also R32.1, U$1.(ADC2:0/TOUCH0/RTC10/SPIHD)GPIO4; no longer T2-2.G
- net GND: now also ACC.1, C28.1, C29.1, C30.2, C31.2, FT231X.GND, IC1.GND, IC2.GND, M365_CONNECTOR.4, R14.1, R24.1, R25.2, R28.1, R29.1, R31.2, REG.GND, T3-1.S, U$11.GND, USB.GND, USB.SHIELD; no longer ACCEL.1, J1.4, J2.GND, J2.SHIELD, U$2.GND, U$7.GND
- net LED_EN: now also R29.2, U$1.(ADC2:2/TOUCH2/RTC12/SPIWP)GPIO2
- net N$2: now also U$10.1; no longer Q1.1
- net N$3: now also R23.2, R26.1; no longer R1.2, TX1.A
- net N$4: now also C28.2, R1.2, U$1.VDET_2(GPI35/ADC1:7); no longer R2.2, RX1.A
- net N$6: now also FT231X.!RESET, FT231X.3V3OUT, FT231X.VCCIO; no longer U$2.!RESET, U$2.3V3OUT, U$2.VCCIO
- net RX0: now also FT231X.TXD; no longer U$2.TXD
- net TX0: now also FT231X.RXD; no longer U$2.RXD
- net USB-DATA_M: now also USB.D-; no longer J2.D-
- net USB-DATA_P: now also USB.D+; no longer J2.D+
- net USBDM: now also FT231X.USBDM; no longer U$2.USBDM
- net USBDP: now also FT231X.USBDP; no longer U$2.USBDP
Other:
- moved on the sheet: BRK, C1, R1, R2

Commit message: Updated dashboard PCB design. Replaced ESP32-D0DW with ESP32-PicoD4 Added bigger buzzer footprint Removed RGB led
Parts:
- removed C20: 0.1uF, eagle-ltspice:CC0402
- removed C23, C24: 20pF, resistor:C-EUC0402
- removed D2: SMAFJ75A, my-lib:SMAFJ75A
- removed M365_CONNECTOR: (no value), SparkFun-Connectors:CONN_05PTH_LONGPADS
- removed R22, R26, R27: 37.4R, eagle-ltspice:RR0402
- removed R23: 86.6R, eagle-ltspice:RR0402
- removed U$10: X321532768KGB2SI, my-lib:X321532768KGB2SI
- removed U$7: Z3535RGBA, my-lib:Z3535RGBA
- added D6, D7: BAS516,115, BAS516_115:BAS516,115
- added IC3: UNEXPECTEDMAKER_ESP32-PICO-D4, m365_esp32:UNEXPECTEDMAKER_ESP32-PICO-D4
- added M365: (no value), SparkFun-Connectors:CONN_06LONGPADS
- added RED_POWER_LED: (no value), Wurth_Elektronik_Optoelectronics_rev18a:WL-SMCD_0603_150060BS55040
- added U$6: ZL-YDW2722-2705PF-12.5ZL-YDW2722-2705PF-12.5, my-lib:ZL-YDW2722-2705PF-12.5ZL-YDW2722-2705PF-12.5
- C19: value 0.1uF -> (none)
- D1: value SMAFJ75A -> BAS516,115; device my-lib:SMAFJ75A -> BAS516_115:BAS516,115
- R18: value 60.4R -> 300R
- R19: value 37.4R -> 866k
- R20: value 86.6R -> 866k
- R21: value 60.4R -> ??; device eagle-ltspice:RR0402 -> eagle-ltspice:R
- R6: value 715k -> 787k
- U$1: value ESP32 -> TL3302BF260QJ; device esp32:ESP32 -> my-lib:TL3302BF260QJ
- U$2: value Z3535RGBA -> TL3302BF260QJ; device my-lib:Z3535RGBA -> my-lib:TL3302BF260QJ
Connections:
- removed net 32K_XP: C23.1, U$1.32K_XP(GPIO32/ADC1:4/TOUCH9/RTC9), U$10.2
- removed net LIGHT_SENS: C30.1, LS1.2, R28.2, U$1.SENSOR_VN(GPI39/ADC1:3/RTC3)
- removed net LL_B: R21.1, U$1.(GPIO6/SPICLK/HS1_CLK/U1CTS)SD_CLK
- removed net LL_G: R22.1, U$1.(GPIO7/SPI1/HS1_DATA0)SD_DATA0
- removed net LL_R: R23.1, U$1.(GPIO8/SPID/HS1_DATA1)SD_DATA1
- removed net LR_B: R18.1, U$1.(GPIO11/SPICSO/HS1_CMD/U1RTS)SD_CMD
- removed net LR_G: R19.1, U$1.(GPIO10/SPIWP/HS1_DATA3/U1TX)SD_DATA3
- removed net LR_R: R20.1, U$1.(GPIO9/SPIHD/HS1_DATA2/U1RX)SD_DATA2
- removed net N$16: C29.2, R2.2, U$1.SENSOR_CAPN(GPI38/ADC1:2/RTC2)
- removed net N$18: R21.2, U$7.BLUE
- removed net N$19: R22.2, U$7.GREEN
- removed net N$20: R26.2, U$7.RED
- removed net N$21: R18.2, U$2.BLUE
- removed net N$22: R19.2, U$2.GREEN
- removed net N$23: U$1.(VSPIHD/HS2_CMD)GPIO21
- removed net N$25: R27.2, U$2.RED
- removed net N$26: R20.2, R27.1
- removed net N$27: U$1.(VSPIWP/HS2_CLK)GPIO22
- removed net RESET: U$1.CHIP_PU, UMH3N1.DTR1_C
- new net ENABLE: C18.1, IC3G$1.EN, R19.2, U$2.P$1, UMH3N1.DTR2_C
- new net GPIO15_NOT_USED: IC3G$1.IO15
- new net GPIO35: C28.2, IC3G$1.IO35, R1.2
- new net GPIO38: C29.2, IC3G$1.SENSOR_CAPN, R2.2
- new net INTERNAL_FLASH_CLK: IC3G$1.CLK
- new net INTERNAL_FLASH_CMD: IC3G$1.CMD
- new net INTERNAL_FLASH_GPIO16: IC3G$1.IO16
- new net INTERNAL_FLASH_GPIO17: IC3G$1.IO17
- new net INTERNAL_FLASH_SD0: IC3G$1.SD0
- new net INTERNAL_FLASH_SD1: IC3G$1.SD1
- new net SENSOR_VN: C30.1, IC3G$1.SENSOR_VN, LS1.2, R28.2
- new net VDD_SDIO: IC3G$1.VDD_SDIO_NC
- net !TFTRST: now also IC3G$1.IO25; no longer U$1.(DAC1/ADC2:8/RTC6)GPIO25
- net 3V3: now also D6.1, IC3G$1.VDD3P3_CPU, IC3G$1.VDD3P3_RTC, IC3G$1.VDDA, IC3G$1.VDDA3P3_1, IC3G$1.VDDA_2, IC3G$1.VDDA_3, IC3G$1.VDDA_3P3, PROG.3, R19.1, RED_POWER_LED.A; no longer C18.1, C19.1, C20.1, D2.CATHODE, U$1.VDD3P3_CPU, U$1.VDD3P3_RTC, U$1.VDDA, U$1.VDDA3P3, U$2.VCC, U$7.VCC
- net 42V: now also M365.6; no longer M365_CONNECTOR.5
- net 5V: now also D1.1, U$6.+
- net 5V_IN: now also M365.3; no longer M365_CONNECTOR.2
- net 5V_USB: no longer PROG.3
- net BACKLIGHT: now also IC3G$1.IO32; no longer U$1.(GPIO15/ADC2:3/TOUCH3/RTC13/SPICSO/U0RTS)MTDO
- net BTN_CENTER: now also D7.2, IC3G$1.SD3; no longer D1.ANODE, U$1.(VSPICS0/HS1_DATA6)GPIO5
- net BTN_CONTROL: now also IC3G$1.IO21
- net BTN_DOWN: now also IC3G$1.IO18; no longer U$1.(VSPICLK/HS1_DATA7)GPIO18
- net BTN_LEFT: now also IC3G$1.SD2; no longer U$1.(HS1_DATA5)GPIO17
- net BTN_RIGHT: now also IC3G$1.IO4; no longer U$1.(HS1_DATA4)GPIO16
- net BTN_UP: now also IC3G$1.IO23; no longer U$1.GPIO23
- net BUZZER: now also IC3G$1.IO2; no longer U$1.(ADC2:0/TOUCH0/RTC10/SPIHD)GPIO4
- net DC: now also IC3G$1.IO26; no longer U$1.(DAC2/ADC2:9/RTC7)GPIO26
- net GND: now also IC3G$2.GNDPAD, M365.5, R18.1, R20.1, U$1.P$2, U$2.P$2; no longer C19.2, C20.2, C23.2, C24.2, M365_CONNECTOR.4, U$1.GND
- net GPIO0: now also IC3G$1.IO0, U$1.P$1, UMH3N1.DTR1_C; no longer U$1.(ADC2:1/TOUCH1/RTC11/CLK_OUT1)GPIO0, UMH3N1.DTR2_C
- net LED_EN: now also IC3G$1.IO12; no longer U$1.(ADC2:2/TOUCH2/RTC12/SPIWP)GPIO2
- net LNA_IN: now also C19.2, IC3G$1.LNA_IN; no longer ANT1.1, U$1.LNA_IN
- net M365_DATA: now also M365.4; no longer M365_CONNECTOR.3
- net M365_DATA_3V3: now also IC3G$1.IO19; no longer U$1.(VSPID/HS2_DATA3)GPIO20
- net M365_LED_DATA: now also M365.2; no longer M365_CONNECTOR.1
- net M365_LED_DATA_3V3: now also IC3G$1.IO13; no longer U$1.(GPIO13/ADC2:4/TOUCH4/RTC14/SPID/U0CTS)MTCK
- net MOSI: now also IC3G$1.IO14; no longer U$1.(ADC2:7/TOUCH7/RTC17)GPIO27
- net N$1: now also IC3G$1.U0TXD; no longer U$1.(GPIO1/CLK_OUT3/HS2_DATA1)U0TXD
- net N$11: now also D1.2, D6.2, R21.2, U$6.-, U$8.-; no longer CENTER.P$1, D1.CATHODE, T1-2.S
- net N$12: now also R21.1; no longer D2.ANODE, U$8.-
- net N$17: now also IC3G$1.IO22; no longer U$1.(VSPIQ/HS2_DATA2)GPIO19
- net N$2: now also ANT1.1, C19.1; no longer C24.1, U$1.32K_XN(GPIO33/ADC1:5/TOUCH8/RTC8), U$10.1
- net N$29: now also R20.2
- net N$3: now also R18.2, RED_POWER_LED.C; no longer R23.2, R26.1
- net N$4: now also CENTER.P$1, D7.1, T1-2.S; no longer C28.2, R1.2, U$1.VDET_2(GPI35/ADC1:7)
- net RX0: now also IC3G$1.U0RXD; no longer U$1.(GPIO3/CLK_OUT2/HS2_DATA0)U0RXD
- net SCK: now also IC3G$1.IO27; no longer U$1.(GPIO14/ADC2:6/TOUCH6/RTC16/SPICLK)MTMS
- net TFTCS: now also IC3G$1.IO33; no longer U$1.(GPIO12/ADC2:5/TOUCH5/RTC15/SPIQ)MTDI
Other:
- note added: "Near ESP32"
- note removed: "Near VDA"
- note removed: "Near VDA3P3"
- note removed: "Near VDD3P3_CPU"
- note removed: "Near VDD3P3_RTC"
- moved on the sheet: ACC, ANT1, BRK, C16, C17, C18, C19, C25, C26, C28, C29, C30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
